File: Conformal Switching Regulator/Kicad Files/ConformalRef/ConformalPowerCircuit.kicad_sch (KiCad schematic)
At the start: 12 parts, among them IC4 TPS54627DDAR

Commit message: BOM
Parts:
- C10, C11, C12, C13, C14, C15, C16, R15, R16, R17: MPN (none) -> Generic
- IC4: MPN (none) -> TPS54627DDAR
- L3: MPN (none) -> IHLP2525BDER1R5M01
